Commit message: update

File: robot_model/urdf/my_robot.urdf (robot description, URDF)
Before this commit: robot ros2_robot, 7 links, 6 joints
Links:
- added link camera_link, mass 5.0; collision box size=0.05 0.05 0.05; visual box size=0.05 0.05 0.05
- link lidar_link: mass 1.0 -> 1e-5
Joints:
- added joint camera_joint: type fixed, parent base_link, child camera_link, origin xyz=0.32 0.0 0.07 rpy=0.0 0.0 0.0, axis 0.0 0.0 0.0, limit lower=0.0 upper=0.0 effort=0.0 velocity=0.0
- joint back_left_joint: limit lower=0.0 upper=0.0 effort=0.0 velocity=0.0 -> lower=0.0 upper=0.0 effort=10.0 velocity=10.0
- joint back_right_joint: limit lower=0.0 upper=0.0 effort=0.0 velocity=0.0 -> lower=0.0 upper=0.0 effort=10.0 velocity=10.0
- joint front_left_joint: limit lower=0.0 upper=0.0 effort=0.0 velocity=0.0 -> lower=0.0 upper=0.0 effort=10.0 velocity=10.0
- joint front_right_joint: limit lower=0.0 upper=0.0 effort=0.0 velocity=0.0 -> lower=0.0 upper=0.0 effort=10.0 velocity=10.0
- joint lidar_joint: axis 0.0 1.0 0.0 -> 0.0 0.0 0.0
